File: hardware/Z280-SBC/Z280-SBC.kicad_pcb (KiCad board)
At the start: 2 copper layers, 308.6 x 160 mm, 96 parts, among them J1 CompactFlash, J2 Serial1, J3 POWER, J4 ATF-JTAG-10, J5 Conn_02x10_Odd_Even, J6 ADBUS, J7 SIGBUS, Q1 2N7002, SW1 RESET, U1 74HC14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

Commit message: Work in progress on PCB design, address and data buses mostly connected
Parts:
- removed the C1 at (309.9, 205.7)
- removed the C10 at (304.8, 127.0)
- removed the C11 at (330.2, 119.4)
- removed the C12 at (431.8, 180.3)
- removed the C13 at (447.0, 180.3)
- removed the C14 at (449.6, 193.0)
- removed the C15 at (330.2, 150.8)
- removed the C16 at (411.5, 180.3)
- removed the C2 at (401.3, 226.5)
- removed the C3 at (408.9, 226.1)
- removed the C4 at (406.4, 149.9)
- removed the C5 at (406.4, 160.0)
- removed the C6 at (414.0, 193.0)
- removed the C7 at (414.0, 205.7)
- removed the C8 at (429.3, 193.0)
- removed the C9 at (407.4, 154.9)
- removed the J1 at (330.2, 61.0)
- removed the J2 at (317.5, 104.1)
- removed the J3 at (297.2, 127.0)
- removed the J4 at (345.4, 39.4)
- removed the J5 at (395.0, 39.4)
- removed the J6 at (395.0, 129.5)
- removed the J7 at (395.0, 71.1)
- removed the JP1 at (410.8, 142.2)
- removed the JP2 at (419.1, 144.8)
- removed the JP3 at (428.3, 135.7)
- removed the JP4 at (420.4, 139.5)
- removed the JP5 at (449.6, 167.6)
- removed the JP6 at (317.5, 115.6)
- removed the Q1 at (416.6, 185.4)
- removed the R1 at (309.9, 210.8)
- removed the R2 at (298.4, 198.8)
- removed the R3 at (416.6, 170.2)
- removed the R4 at (406.4, 170.2)
- removed the RN1 at (330.2, 145.8)
- removed the SW1 at (299.0, 206.0)
- removed the U1 at (362.9, 99.1)
- removed the U10 at (360.7, 50.8)
- removed the U2 at (360.7, 121.9)
- removed the U3 at (335.3, 163.8)
- removed the U4 at (335.3, 176.5)
- removed the U5 at (373.4, 106.7)
- removed the U6 at (352.7, 101.6)
- removed the U7 at (373.4, 168.9)
- removed the U8 at (351.0, 168.7)
- removed the U9 at (337.8, 101.6)
- removed the Y1 at (403.9, 221.0)
- removed the Y2 at (411.5, 175.3)
- added J8: IE/OE, Connector_PinHeader_2.54mm:PinHeader_1x02_P2.54mm_Vertical, F.Cu at (134.6, 34.3)
- J5: value Conn_02x10_Odd_Even -> COUNTER1; footprint Connector_PinHeader_2.54mm:PinHeader_2x10_P2.54mm_Vertical -> Connector_PinHeader_2.54mm:PinHeader_1x02_P2.54mm_Vertical
- U10: value ATF1504AS-10JU84 -> ATF1504AS-xJx44; footprint Package_LCC:PLCC-84_THT-Socket -> Package_LCC:PLCC-44_THT-Socket
- moved JP3 150.1 mm to (55.9, 30.5), turned to 180 degrees
- moved C14 141.8 mm to (90.9, 149.7)
- moved JP2 141.6 mm to (55.9, 35.6), turned to 180 degrees
- moved JP4 141.5 mm to (55.9, 40.8), turned to 180 degrees
- moved JP1 131.8 mm to (55.9, 45.7), turned to 180 degrees
- moved J2 131.4 mm to (56.4, 51.3), turned to 0 degrees
- moved C3 130.7 mm to (109.2, 33.5), turned to 180 degrees
- moved C2 123.3 mm to (116.8, 33.0), turned to 180 degrees
- moved C12 120.8 mm to (87.6, 88.9), turned to 180 degrees
- moved U5 116.9 mm to (101.6, 94.3)
- moved Y1 116.5 mm to (114.3, 38.6), turned to 180 degrees
- moved JP6 114.1 mm to (62.2, 58.4), turned to 0 degrees
- moved C13 113.6 mm to (112.5, 118.4), turned to -90 degrees
- moved J5 111.1 mm to (125.7, 34.3)
- moved C16 109.9 mm to (90.8, 145.3)
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Connections:
- J5 pad 1: unconnected-(J5-Pad1) -> CTIN1
- J5 pad 2: CTIN1 -> CTIO1
- J7 pad 16: unconnected-(J7-Pad16) -> B/~{W}
- J7 pad 19: ROMSEL -> ~{ROMSEL}
- J7 pad 21: 0SEL -> ~{0SEL}
- J7 pad 23: RAMSEL -> ~{RAMSEL}
- J7 pad 25: 2SEL -> ~{2SEL}
- J7 pad 27: 3SEL -> ~{3SEL}
- J7 pad 29: 4SEL -> ~{4SEL}
- J7 pad 31: 5SEL -> ~{5SEL}
- J7 pad 33: 6SEL -> ~{6SEL}
- J7 pad 34: GPIO1 -> CTIN2
- J7 pad 35: IOSEL -> ~{IOSEL}
- J7 pad 36: GPIO2 -> CTIO2
- J7 pad 38: GPIO3 -> ~{AOE}
- J7 pad 7: GPIO4 -> unconnected-(J7-Pad7)
- R2 pad 2: ~{GREQ} -> ~{RESET}
- R4 pad 1: BACKUP_CLK -> ALT_CLK
- RN1 pad 2: ~{RESET} -> ~{WAIT}
- RN1 pad 3: ~{WAIT} -> ~{PAUSE}
- RN1 pad 4: ~{PAUSE} -> ~{BUSREQ}
- RN1 pad 5: ~{BUSREQ} -> ~{GREQ}
- U1 pad 12: BACKUP_CLK -> ALT_CLK
- U10 pad 1: unconnected-(U10-Pad1) -> CTIN2
- U10 pad 10: BACKUP_CLK -> GND
- U10 pad 11: ~{RESET} -> ~{AS}
- U10 pad 12: ~{WAIT} -> ~{DS}
- U10 pad 13: +5V -> Net-(J4-Pad5)
- U10 pad 14: Net-(J4-Pad9) -> B/~{W}
- U10 pad 15: ~{PAUSE} -> +5V
- U10 pad 16: ~{AS} -> R/~{W}
- U10 pad 17: ~{DS} -> ST0
- U10 pad 18: B/~{W} -> ST1
- U10 pad 19: GND -> ST2
- U10 pad 2: unconnected-(U10-Pad2) -> ALT_CLK
- U10 pad 20: R/~{W} -> ST3
- U10 pad 21: ~{IE} -> ATA-READY
- U10 pad 22: ~{OE} -> GND
- U10 pad 23: Net-(J4-Pad5) -> +5V
- U10 pad 24: ST0 -> ~{NMI}
- U10 pad 25: ST1 -> ~{INTc}
- U10 pad 26: +5V -> ~{INTb}
- U10 pad 27: ST2 -> ~{INTa}
- U10 pad 28: ST3 -> A23
- U10 pad 29: ~{UDS} -> A22
- U10 pad 30: ~{LDS} -> GND
- U10 pad 31: unconnected-(U10-Pad31) -> A21
- U10 pad 32: GND -> Net-(J4-Pad1)
- U10 pad 33: unconnected-(U10-Pad33) -> ~{GREQ}
- U10 pad 34: unconnected-(U10-Pad34) -> ~{GACK}
- U10 pad 35: unconnected-(U10-Pad35) -> +5V
- U10 pad 36: unconnected-(U10-Pad36) -> ~{BUSACK}
- U10 pad 37: unconnected-(U10-Pad37) -> ~{BUSREQ}
- U10 pad 38: +5V -> Net-(J4-Pad3)
- U10 pad 39: unconnected-(U10-Pad39) -> ROMSEL
- U10 pad 4: ~{INTa} -> CTIO2
- U10 pad 40: unconnected-(U10-Pad40) -> ~{RAMSEL}
- U10 pad 41: unconnected-(U10-Pad41) -> CTIO1
- U10 pad 43: +5V -> CLK
- U10 pad 44: unconnected-(U10-Pad44) -> CTIN1
- U10 pad 5: ~{INTb} -> ~{AOE}
- U10 pad 6: ~{INTc} -> ~{RESET}
- U10 pad 7: GND -> Net-(J4-Pad9)
- U10 pad 8: ~{NMI} -> ~{WAIT}
- U10 pad 9: CLK -> ~{PAUSE}
- Y2 pad 2: BACKUP_CLK -> ALT_CLK
Routing:
- net D7: track 0.00 -> 140.9 mm, vias 0 -> 6
- net A19: track 0.00 -> 139.0 mm, vias 0 -> 4
- net D9: track 0.00 -> 135.0 mm, vias 0 -> 3
- net D11: track 0.00 -> 134.0 mm, vias 0 -> 3
- net A18: track 0.00 -> 132.9 mm, vias 0 -> 4
- net D6: track 0.00 -> 132.7 mm, vias 0 -> 6
- net D8: track 0.00 -> 132.6 mm, vias 0 -> 3
- net D10: track 0.00 -> 131.3 mm, vias 0 -> 3
- net A17: track 0.00 -> 128.4 mm, vias 0 -> 3
- net D4: track 0.00 -> 128.3 mm, vias 0 -> 6
- net D13: track 0.00 -> 128.3 mm, vias 0 -> 3
- net D5: track 0.00 -> 128.1 mm, vias 0 -> 6
- net D15: track 0.00 -> 127.2 mm, vias 0 -> 3
- net D14: track 0.00 -> 126.9 mm, vias 0 -> 3
- net A16: track 0.00 -> 126.7 mm, vias 0 -> 3
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Other:
- board size 308.6 x 160 mm -> 100 x 160 mm

Commit message: Mostly done Rev1
Parts:
- added J10: POWER, Connector_PinHeader_2.54mm:PinHeader_1x02_P2.54mm_Vertical, F.Cu at (70.4, 140.1)
- added J9: POWER, Connector_PinHeader_2.54mm:PinHeader_1x02_P2.54mm_Vertical, F.Cu at (66.3, 140.1)
- added REF**: OSHW-Symbol_6.7x6mm_SilkScreen, Symbol:OSHW-Symbol_6.7x6mm_SilkScreen, F.Cu at (86.4, 129.3)
- moved C14 91.8 mm to (81.3, 58.4)
- moved C16 89.1 mm to (71.1, 58.4)
- moved JP3 84.3 mm to (89.2, 108.0)
- moved JP1 79.7 mm to (89.2, 118.1), turned to 0 degrees
- moved JP4 79.6 mm to (89.2, 113.2)
- moved JP2 75.1 mm to (89.2, 102.9)
- moved J8 26.7 mm to (108.0, 36.2)
- moved C1 25.0 mm to (56.0, 130.0), turned to 180 degrees
- moved J3 24.8 mm to (74.4, 140.1), turned to 180 degrees
- moved R1 22.8 mm to (59.9, 140.2)
- moved J5 22.3 mm to (103.5, 36.2)
- moved SW1 20.5 mm to (52.6, 140.9)
- moved Y1 17.8 mm to (132.1, 38.1)
- moved C3 17.8 mm to (127.0, 33.0)
- moved C2 15.4 mm to (132.2, 33.0), turned to 0 degrees
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Connections:
- JP5 pad 1: 0SEL -> ~{0SEL}
- JP5 pad 2: ROMSEL -> ~{ROMSEL}
- JP5 pad 3: 2SEL -> ~{2SEL}
Routing:
- net ~{AOE}: track 0.00 -> 178.9 mm, vias 0 -> 4
- net R~{W}: track 0.00 -> 176.1 mm, vias 0 -> 5
- net ~{PAUSE}: track 0.00 -> 148.1 mm, vias 0 -> 4
- net ~{WAIT}: track 0.00 -> 146.6 mm, vias 0 -> 4
- net ~{BUSACK}: track 0.00 -> 140.2 mm, vias 0 -> 4
- net ~{AS}: track 0.00 -> 137.4 mm, vias 0 -> 3
- net ~{RAMSEL}: track 0.00 -> 127.9 mm, vias 0 -> 4
- net ~{RESET}: track 0.00 -> 123.9 mm, vias 0 -> 4
- net GND: track 0.00 -> 120.3 mm, vias 0 -> 23
- net ~{BUSREQ}: track 0.00 -> 120.3 mm, vias 0 -> 4
- net ~{GREQ}: track 0.00 -> 109.4 mm, vias 0 -> 6
- net ~{DS}: track 0.00 -> 97.5 mm, vias 0 -> 4
- net ~{ROMSEL}: track 0.00 -> 81.7 mm, vias 0 -> 3
- net ~{6SEL}: track 0.00 -> 78.4 mm, vias 0 -> 3
- net ~{0SEL}: track 0.00 -> 71.5 mm, vias 0 -> 1
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- added copper zone on In1.Cu, net +5V
- added copper zone on B.Cu, net GND
- added copper zone on F.Cu, net GND
- added copper zone on In2.Cu, net GND
Other:
- board size 100 x 160 mm -> 100 x 115 mm
- copper layers 2 -> 4
- board text added: "Designed by transistor fet 2022"
- board text added: "Z280-SBC Rev. 1"
