File: hardware/Z280-SBC/Z280-SBC.kicad_sch (KiCad schematic)
At the start: 17 parts, among them Q1 2N7002, SW1 RESET, U1 74HC14, U2 Z280CPU, U3 74HC573, U4 74HC573, Y1 Crystal, Y2 Crystal

Commit message: Work in progress on PCB design, address and data buses mostly connected
Connections:
- net ~{BUSREQ}: now also RN1.4 (R3); no longer RN1.5 (R4)
- net ~{GREQ}: now also RN1.5 (R4); no longer R2.2
- net ~{PAUSE}: now also RN1.3 (R2); no longer RN1.4 (R3)
- net ~{RESET}: now also R2.2; no longer RN1.2 (R1)
- net ~{WAIT}: now also RN1.2 (R1); no longer RN1.3 (R2)
- net BACKUP_CLK renamed ALT_CLK
Other:
- moved on the sheet: R2

Commit message: Rev1 - All connections completed
Connections:
- net ~{INTc}: now reaches RN1.6 (R5), U2.26 (~{INTc})
- net ~{INTb}: now reaches RN1.7 (R6), U2.36 (~{INTb/EOPb})
- net ~{INTa}: now reaches RN1.8 (R7), U2.37 (~{INTa/EOPa})
- net ~{NMI}: now reaches RN1.9 (R8), U2.39 (~{NMI})
- net R~{W} renamed R/~{W}
Changed lines of the file:
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@@
   (junction (at 81.28 31.75) (diameter 0) (color 0 0 0 0)
   )
+  (junction (at 69.85 50.8) (diameter 0) (color 0 0 0 0)
+  )
   (junction (at 35.56 167.64) (diameter 0) (color 0 0 0 0)
   )
@@
   (junction (at 62.23 119.38) (diameter 0) (color 0 0 0 0)
   )
+  (junction (at 67.31 53.34) (diameter 0) (color 0 0 0 0)
+  )
   (junction (at 109.22 135.89) (diameter 0) (color 0 0 0 0)
   )
+  (junction (at 64.77 55.88) (diameter 0) (color 0 0 0 0)
+  )
   (junction (at 49.53 66.04) (diameter 0) (color 0 0 0 0)
   )
@@
   )
   (junction (at 125.73 170.18) (diameter 0) (color 0 0 0 0)
+  )
+  (junction (at 72.39 48.26) (diameter 0) (color 0 0 0 0)
   )
   (junction (at 140.97 170.18) (diameter 0) (color 0 0 0 0)
@@
     (stroke (width 0) (type default) (color 0 0 0 0))
   )
+  (wire (pts (xy 44.45 55.88) (xy 64.77 55.88))
+    (stroke (width 0) (type default) (color 0 0 0 0))
+  )
   (wire (pts (xy 140.97 180.34) (xy 140.97 170.18))
     (stroke (width 0) (type default) (color 0 0 0 0))
@@
     (stroke (width 0) (type default) (color 0 0 0 0))
   )
-  (wire (pts (xy 48.26 78.74) (xy 90.17 78.74))
+  (wire (pts (xy 44.45 78.74) (xy 90.17 78.74))
     (stroke (width 0) (type default) (color 0 0 0 0))
   )
@@
     (stroke (width 0) (type default) (color 0 0 0 0))
   )
-  (wire (pts (xy 48.26 68.58) (xy 54.61 68.58))
+  (wire (pts (xy 44.45 68.58) (xy 54.61 68.58))
     (stroke (width 0) (type default) (color 0 0 0 0))
   )
@@
     (stroke (width 0) (type default) (color 0 0 0 0))
   )
-  (wire (pts (xy 64.77 55.88) (xy 64.77 41.91))
+  (wire (pts (xy 44.45 48.26) (xy 72.39 48.26))
     (stroke (width 0) (type default) (color 0 0 0 0))
   )
@@
     (stroke (width 0) (type default) (color 0 0 0 0))
   )
+  (wire (pts (xy 44.45 53.34) (xy 67.31 53.34))
+    (stroke (width 0) (type default) (color 0 0 0 0))
+  )
   (wire (pts (xy 208.28 40.64) (xy 220.98 40.64))
     (stroke (width 0) (type default) (color 0 0 0 0))
@@
     (stroke (width 0) (type default) (color 0 0 0 0))
   )
-  (wire (pts (xy 48.26 73.66) (xy 90.17 73.66))
+  (wire (pts (xy 44.45 73.66) (xy 90.17 73.66))
     (stroke (width 0) (type default) (color 0 0 0 0))
   )
@@
     (stroke (width 0) (type default) (color 0 0 0 0))
   )
-  (wire (pts (xy 48.26 76.2) (xy 90.17 76.2))
+  (wire (pts (xy 44.45 76.2) (xy 90.17 76.2))
     (stroke (width 0) (type default) (color 0 0 0 0))
   )
@@
     (stroke (width 0) (type default) (color 0 0 0 0))
   )
-  (wire (pts (xy 48.26 66.04) (xy 49.53 66.04))
+  (wire (pts (xy 44.45 66.04) (xy 49.53 66.04))
     (stroke (width 0) (type default) (color 0 0 0 0))
   )
@@
     (stroke (width 0) (type default) (color 0 0 0 0))
   )
+  (wire (pts (xy 64.77 41.91) (xy 64.77 55.88))
+    (stroke (width 0) (type default) (color 0 0 0 0))
+  )
   (wire (pts (xy 196.85 58.42) (xy 189.23 58.42))
     (stroke (width 0) (type default) (color 0 0 0 0))
@@
     (stroke (width 0) (type default) (color 0 0 0 0))
   )
+  (wire (pts (xy 44.45 50.8) (xy 69.85 50.8))
+    (stroke (width 0) (type default) (color 0 0 0 0))
+  )
   (wire (pts (xy 189.23 90.17) (xy 196.85 90.17))
     (stroke (width 0) (type default) (color 0 0 0 0))
@@
     (stroke (width 0) (type default) (color 0 0 0 0))
   )
-  (wire (pts (xy 48.26 71.12) (xy 57.15 71.12))
+  (wire (pts (xy 44.45 71.12) (xy 57.15 71.12))
     (stroke (width 0) (type default) (color 0 0 0 0))
   )
@@
     )
   )
-  (global_label "R~{W}" (shape output) (at 20.32 91.44 180) (fields_autoplaced)
-    (effects (font (size 1.27 1.27)) (justify right))
-    (property "Intersheet References" "${INTERSHEET_REFS}" (id 0) (at 218.44 -68.58 0)
-      (effects (font (size 1.27 1.27)) (justify left) hide)
-    )
-  )
-  (global_label "B{slash}~{W}" (shape output) (at 48.26 78.74 180) (fields_autoplaced)
-    (effects (font (size 1.27 1.27)) (justify right))
-    (property "Intersheet References" "${INTERSHEET_REFS}" (id 0) (at 41.795 78.6606 0)
+  (global_label "R{slash}~{W}" (shape output) (at 20.32 91.44 180) (fields_autoplaced)
+    (effects (font (size 1.27 1.27)) (justify right))
+    (property "Intersheet References" "${INTERSHEET_REFS}" (id 0) (at 13.855 91.3606 0)
+      (effects (font (size 1.27 1.27)) (justify right) hide)
+    )
+  )
+  (global_label "B{slash}~{W}" (shape output) (at 44.45 78.74 180) (fields_autoplaced)
+    (effects (font (size 1.27 1.27)) (justify right))
+    (property "Intersheet References" "${INTERSHEET_REFS}" (id 0) (at 37.985 78.6606 0)
+      (effects (font (size 1.27 1.27)) (justify right) hide)
+    )
+  )
+  (global_label "~{INTb}" (shape input) (at 44.45 53.34 180) (fields_autoplaced)
+    (effects (font (size 1.27 1.27)) (justify right))
+    (property "Intersheet References" "${INTERSHEET_REFS}" (id 0) (at 37.985 53.2606 0)
       (effects (font (size 1.27 1.27)) (justify right) hide)
     )
@@
     )
   )
+  (global_label "~{INTa}" (shape input) (at 44.45 50.8 180) (fields_autoplaced)
+    (effects (font (size 1.27 1.27)) (justify right))
+    (property "Intersheet References" "${INTERSHEET_REFS}" (id 0) (at 37.985 50.7206 0)
+      (effects (font (size 1.27 1.27)) (justify right) hide)
+    )
+  )
+  (global_label "~{INTc}" (shape input) (at 44.45 55.88 180) (fields_autoplaced)
+    (effects (font (size 1.27 1.27)) (justify right))
+    (property "Intersheet References" "${INTERSHEET_REFS}" (id 0) (at 38.0455 55.8006 0)
+      (effects (font (size 1.27 1.27)) (justify right) hide)
+    )
+  )
   (global_label "~{AS}" (shape input) (at 161.29 107.95 180) (fields_autoplaced)
     (effects (font (size 1.27 1.27)) (justify right))
@@
     )
   )
-  (global_label "~{WAIT}" (shape input) (at 48.26 68.58 180) (fields_autoplaced)
-    (effects (font (size 1.27 1.27)) (justify right))
-    (property "Intersheet References" "${INTERSHEET_REFS}" (id 0) (at 41.7345 68.5006 0)
-      (effects (font (size 1.27 1.27)) (justify right) hide)
-    )
-  )
-  (global_label "~{PAUSE}" (shape input) (at 48.26 71.12 180) (fields_autoplaced)
-    (effects (font (size 1.27 1.27)) (justify right))
-    (property "Intersheet References" "${INTERSHEET_REFS}" (id 0) (at 39.7993 71.0406 0)
+  (global_label "~{WAIT}" (shape input) (at 44.45 68.58 180) (fields_autoplaced)
+    (effects (font (size 1.27 1.27)) (justify right))
+    (property "Intersheet References" "${INTERSHEET_REFS}" (id 0) (at 37.9245 68.5006 0)
+      (effects (font (size 1.27 1.27)) (justify right) hide)
+    )
+  )
+  (global_label "~{PAUSE}" (shape input) (at 44.45 71.12 180) (fields_autoplaced)
+    (effects (font (size 1.27 1.27)) (justify right))
+    (property "Intersheet References" "${INTERSHEET_REFS}" (id 0) (at 35.9893 71.0406 0)
       (effects (font (size 1.27 1.27)) (justify right) hide)
     )
@@
     )
   )
+  (global_label "~{NMI}" (shape input) (at 44.45 48.26 180) (fields_autoplaced)
+    (effects (font (size 1.27 1.27)) (justify right))
+    (property "Intersheet References" "${INTERSHEET_REFS}" (id 0) (at 38.6502 48.1806 0)
+      (effects (font (size 1.27 1.27)) (justify right) hide)
+    )
+  )
   (global_label "CLK" (shape output) (at 82.55 43.18 180) (fields_autoplaced)
     (effects (font (size 1.27 1.27)) (justify right))
@@
     )
   )
-  (global_label "~{DS}" (shape output) (at 48.26 76.2 180) (fields_autoplaced)
-    (effects (font (size 1.27 1.27)) (justify right))
-    (property "Intersheet References" "${INTERSHEET_REFS}" (id 0) (at 43.3674 76.1206 0)
+  (global_label "~{DS}" (shape output) (at 44.45 76.2 180) (fields_autoplaced)
+    (effects (font (size 1.27 1.27)) (justify right))
+    (property "Intersheet References" "${INTERSHEET_REFS}" (id 0) (at 39.5574 76.1206 0)
       (effects (font (size 1.27 1.27)) (justify right) hide)
     )
@@
     )
   )
-  (global_label "~{RESET}" (shape input) (at 48.26 66.04 180) (fields_autoplaced)
-    (effects (font (size 1.27 1.27)) (justify right))
-    (property "Intersheet References" "${INTERSHEET_REFS}" (id 0) (at 40.1017 65.9606 0)
-      (effects (font (size 1.27 1.27)) (justify right) hide)
-    )
-  )
-  (global_label "~{AS}" (shape output) (at 48.26 73.66 180) (fields_autoplaced)
-    (effects (font (size 1.27 1.27)) (justify right))
-    (property "Intersheet References" "${INTERSHEET_REFS}" (id 0) (at 43.5488 73.5806 0)
-      (effects (font (size 1.27 1.27)) (justify right) hide)
-    )
+  (global_label "~{RESET}" (shape input) (at 44.45 66.04 180) (fields_autoplaced)
+    (effects (font (size 1.27 1.27)) (justify right))
+    (property "Intersheet References" "${INTERSHEET_REFS}" (id 0) (at 36.2917 65.9606 0)
+      (effects (font (size 1.27 1.27)) (justify right) hide)
+    )
+  )
+  (global_label "~{AS}" (shape output) (at 44.45 73.66 180) (fields_autoplaced)
+    (effects (font (size 1.27 1.27)) (justify right))
+    (property "Intersheet References" "${INTERSHEET_REFS}" (id 0) (at 39.7388 73.5806 0)
+      (effects (font (size 1.27 1.27)) (justify right) hide)
+    )

Commit message: Z280-SBC Revision 1 is complete
Other:
- title: (none) -> Z280-SBC
Changed lines of the file:
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@@
 (kicad_sch (version 20211123) (generator eeschema)
   (paper "A4")
+  (title_block
+    (title "Z280-SBC")
+    (rev "1")
+  )
   (junction (at 81.28 31.75) (diameter 0) (color 0 0 0 0)
   )
@@
       (reference "C16") (unit 1) (value "0.1uF") (footprint "Capacitor_SMD:C_1206_3216Metric_Pad1.33x1.80mm_HandSolder")
     )
+    (path "/4f5962dd-3951-476e-a642-9dc05aa10c51/727a030f-a21a-408e-a280-dfe450ef17c6"
+      (reference "C17") (unit 1) (value "0.1uF") (footprint "Capacitor_SMD:C_1206_3216Metric_Pad1.33x1.80mm_HandSolder")
+    )
     (path "/4f5962dd-3951-476e-a642-9dc05aa10c51/32ff13e9-2fc8-4451-8008-990360d1c539"
       (reference "J1") (unit 1) (value "CompactFlash") (footprint "Computie_Connectors:CF-Card_3M_N7E50-Q516RB-40")
@@
     )
     (path "/90e9c810-888d-48c4-9c9e-639527fe4c40/1cdfe995-09d1-49cd-b2e9-94d54f942738"
-      (reference "U7") (unit 1) (value "M29F800") (footprint "Package_SO:TSOP-I-48_18.4x12mm_P0.5mm")
+      (reference "U7") (unit 1) (value "M29F160") (footprint "Package_SO:TSOP-I-48_18.4x12mm_P0.5mm")
     )
     (path "/90e9c810-888d-48c4-9c9e-639527fe4c40/c4f74494-570d-402f-8056-6372acc55fdd"
