File: hardware/Z280-SBC/Bus.kicad_sch (KiCad schematic)
At the start: 6 parts, among them J4 ATF-JTAG-10, J5 COUNTER1, J6 ADBUS, J7 SIGBUS, J8 IE/OE, U10 ATF1504AS-xJx44

Commit message: Added computie-kicad-library and fixed references to point to it
Parts:
- U10: symbol Z280:ATF1504AS-xJx44 -> Computie_CPLDs:ATF1504AS-xJx44
