File: hardware/Z280-SBC/IO.kicad_sch (KiCad schematic)
At the start: 20 parts, among them J1 CompactFlash, J2 Serial1, J3 POWER, U1 74HC14, U6 74HC08, U9 74HC32

Commit message: Mostly done Rev1
Parts:
- added J10, J9: POWER, Connector_PinHeader_2.54mm:PinHeader_1x02_P2.54mm_Vertical, symbol Connector_Generic:Conn_01x02
Connections:
- net +5V: now also J10.1 (Pin_1), J9.1 (Pin_1)
- net GND: now also J10.2 (Pin_2), J9.2 (Pin_2)
Other:
- moved on the sheet: C10, J3

Commit message: Z280-SBC Revision 1 is complete
Parts:
- added C17: 0.1uF, Capacitor_SMD:C_1206_3216Metric_Pad1.33x1.80mm_HandSolder, symbol Device:C_Small
Connections:
- net +5V: now also C17.1
- net GND: now also C17.2
Other:
- title: (none) -> Z280-SBC
- moved on the sheet: C12, C14, C16, C5, C7, C9

Commit message: Fixed most of the issues with Rev.1
Other:
- note added: "COMPACTFLASH CARD SLOT & CONTROL"
- note added: "SERIAL PORT CONNECTION"
Changed lines of the file:
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@@
   (title_block
     (title "Z280-SBC")
-    (rev "1")
+    (rev "2")
   )
   (junction (at 203.2 62.23) (diameter 0) (color 0 0 0 0)
@@
     (stroke (width 0) (type default) (color 0 0 0 0))
   )
+  (text "SERIAL PORT CONNECTION" (at 101.6 25.4 0)
+    (effects (font (size 1.27 1.27) bold italic) (justify left bottom))
+  )
+  (text "COMPACTFLASH CARD SLOT & CONTROL\n" (at 96.52 82.55 0)
+    (effects (font (size 1.27 1.27) bold italic) (justify left bottom))
+  )
   (label "A2" (at 93.98 146.05 0)
